File: PCB Design/PCB Design/PCB Design.sch (EAGLE design)
At the start: 0 parts

Commit message: Completed Schematic, no text module
Parts:
- added J1: 1X2-3.5MM, adafruit:1X2-3.5MM
- added U$1: GPS-RECEIVER-NEO6M, diy-modules:GPS-RECEIVER-NEO6M
- added U$2: SOUND-BUZZER, diy-modules:SOUND-BUZZER
- added U$3: ESP32DEVKITV1, ESP32-DEVKITV1:ESP32DEVKITV1
- added U1: ADXL337, SparkFun-Sensors:ADXL337
Connections:
- new net N$1: U$1.VCC, U$2.VCC, U$3.3V3, U1.VS@1, U1.VS@2
- new net N$10: U$1.TXD, U$3.IO3
- new net N$11: U$2.EN, U$3.IO5
- new net N$2: U$1.GND, U$2.GND, U$3.GND, U1.GND@1, U1.GND@2
- new net N$3: U$3.IO32, U1.ST
- new net N$4: J1.1, U$3.VIN
- new net N$5: J1.2, U$3.GND1
- new net N$6: U$3.IO15, U1.XOUT
- new net N$7: U$3.IO2, U1.YOUT
- new net N$8: U$3.IO4, U1.ZOUT
- new net N$9: U$1.RXD, U$3.IO1
Other:
- note added: "ST should be 0 unless testing functionality"
