File: PCB Design/PCB Design/PCB Design.brd (EAGLE design)
At the start: 120.6 x 88.6 mm, 6 parts, among them J1 1X2-3.5MM, U1 ADXL337

Commit message: added team members names and connection points with labels
Routing:
- net N$6: track 21.1 -> 108.1 mm, vias 1 -> 2
- net N$8: track 23.2 -> 80.2 mm, vias 1 -> 3
- net N$7: track 24.8 -> 80.9 mm, vias 1 -> 3
- net 3.3V: track 81.3 -> 134.2 mm, vias 2 -> 3
- net N$9: track 82.6 -> 122.5 mm, vias 0 -> 1
- net N$10: track 77.9 -> 113.6 mm, vias 0 -> 1
- net GND: vias 0 -> 1
Other:
- board text added: "+3.3V"
- board text added: "ACC-X"
- board text added: "ACC-Y"
- board text added: "ACC-Z"
- board text added: "GND"
- board text added: "GPS-RXD"
- board text added: "GPS-TXT"
- board text added: "Team 14 Hayden Pietsch Amanda Vuong Jaxon Coward Erick I. Cortez Valdez"
